Commit message: removed rendering of the rotors of MAV

File: rotors_description/urdf/multirotor_base.xacro (robot description, xacro)
@@ -89,18 +89,18 @@
         <xacro:insert_block name="inertia" />
       </inertial>
-      <visual>
-        <geometry>
+      <!-- <visual> -->
+        <!-- <geometry> -->
           <!-- <cylinder length="0.005" radius="${radius_rotor}"/> --> <!-- [m] -->
-          <xacro:if value="${use_own_mesh}">
+          <!-- <xacro:if value="${use_own_mesh}">
             <mesh filename="${mesh}"
               scale="1 1 1" />
-          </xacro:if>
-          <xacro:unless value="${use_own_mesh}">
+          </xacro:if> -->
+          <!-- <xacro:unless value="${use_own_mesh}">
             <mesh filename="package://rotors_description/meshes/propeller_${direction}.dae"
-              scale="${radius_rotor} ${radius_rotor} ${radius_rotor}" /> <!-- The propeller meshes have a radius of 1m -->
+              scale="${radius_rotor} ${radius_rotor} ${radius_rotor}" />  -->
             <!-- <box size="${2*radius_rotor} 0.01 0.005"/> -->
-          </xacro:unless>
-        </geometry>
-      </visual>
+          <!-- </xacro:unless> -->
+        <!-- </geometry> -->
+      <!-- </visual> -->
       <collision>
         <geometry>

Commit message: actor with different optional animations. multirotor rotor animations enabled

File: rotors_description/urdf/multirotor_base.xacro (robot description, xacro)
@@ -89,18 +89,18 @@
         <xacro:insert_block name="inertia" />
       </inertial>
-      <!-- <visual> -->
-        <!-- <geometry> -->
+      <visual>
+        <geometry>
           <!-- <cylinder length="0.005" radius="${radius_rotor}"/> --> <!-- [m] -->
-          <!-- <xacro:if value="${use_own_mesh}">
+          <xacro:if value="${use_own_mesh}">
             <mesh filename="${mesh}"
               scale="1 1 1" />
-          </xacro:if> -->
-          <!-- <xacro:unless value="${use_own_mesh}">
+          </xacro:if>
+          <xacro:unless value="${use_own_mesh}">
             <mesh filename="package://rotors_description/meshes/propeller_${direction}.dae"
-              scale="${radius_rotor} ${radius_rotor} ${radius_rotor}" />  -->
+              scale="${radius_rotor} ${radius_rotor} ${radius_rotor}" /> <!-- The propeller meshes have a radius of 1m -->
             <!-- <box size="${2*radius_rotor} 0.01 0.005"/> -->
-          <!-- </xacro:unless> -->
-        <!-- </geometry> -->
-      <!-- </visual> -->
+          </xacro:unless>
+        </geometry>
+      </visual>
       <collision>
         <geometry>
